File: KiCAD/panelone.sch (KiCad schematic (older format))
At the start: 7 parts, among them P1 CONN_AUX3, P2 CONN_AUX2, P4 SD_Header

Commit message: PanelOne v2.0
Warning - Still under development
Parts:
- removed P4: SD_Header, symbol CONN_8
- added C1: 2.2uF, symbol C
- added J1: MICROSD, ~, symbol MICROSD
- added U1: MIC5209-3.3YS, symbol LM7805
- added U2: 4050, symbol 4050
Connections:
- net labels added: +3.3V, CLK, CS, DI, DO, VCC, VI, VO, VSS, _CLK, _CS, _DI
- wire segments 92 -> 121
